File: RASBB/Hardware/Rev.C/Design/RASBB.kicad_pcb (KiCad board)
At the start: 8 copper layers, 167.2 x 95.4 mm, 652 parts, among them IC1 RT6365GSP, IC10 MT41K256M16TW-107_P, IC11 TPD12S016PWR, IC12 STM32H743VGT6, IC13 SX1280IMLTRT, IC14 LAN8742AI-CZ-TR, IC2 TPS56528DDAR, IC3 TPS563201DDCR, IC4 TPS56528DDAR, IC5 S25FL128LAGMFI010, IC6 TS3A5018DBQR, IC7 S25FL128LAGMFI010, IC8 TS3A5018DBQR, IC9 MT41K256M16TW-107_P, J1 PJ-002AH-SMT-TR, J10 ZX-PZ1.27-2-5PWZ, J11 Conn_Coaxial, J12 AudioJack4, J13 Conn_01x06_Socket, J14 HR911196AE, J15 Conn_01x06_Socket, J16 Conn_01x02_Pin, J17 Conn_01x02_Pin, J18 Conn_01x02_Pin, J2 HR911196AE, J3 HDMI-001A, J4 X3157WS-98-9TV30, J5 FH12-50S-0.5SV, J7 USB_C_Receptacle, J8 ZX-PZ1.27-2-5PWZ, J9 KF2EDGR-3.5-2P, Q1 DMN6075S, U1 SZMMSZ4702T1G, U10 XC7A100T-CSG324, U11 XC7A100T-CSG324, U12 RTL8211E-VB-CG, U2 SI2324DS-T1-GE3, U3 SIC453ED-T1-GE3, U4 JW5026, U6 CH340E, U7 AHT20, U8 LM386, U9 LM321, X1 OT2EL4C4JI-111OLP-50M, X3 OT2EL4C4JI-111OLP-50M, X4 OT2EL4C4JI-111OLP-50M, Y1 X503220MSB2GI, Y2 XC21M4-52.000-F10NNHPL, Y3 25MHz

Commit message: Draft AC
Parts:
- added C126: 10nF, Capacitor_SMD:C_0402_1005Metric, F.Cu at (245.8, 82.8)
- added C259: 100nF, Capacitor_SMD:C_0402_1005Metric, F.Cu at (253.5, 82.5)
- added C260: 100nF, Capacitor_SMD:C_0402_1005Metric, F.Cu at (253.5, 79.8)
- added C268: 100nF, Capacitor_SMD:C_0402_1005Metric, F.Cu at (253.5, 81.2)
- added C270: 100nF, Capacitor_SMD:C_0402_1005Metric, B.Cu at (125.4, 108.8)
- added C271: 2200pF, Capacitor_SMD:C_0402_1005Metric, F.Cu at (122.5, 106.8)
- added C272: 2200pF, Capacitor_SMD:C_0402_1005Metric, F.Cu at (125.7, 106.8)
- added C276: 100nF, Capacitor_SMD:C_0402_1005Metric, F.Cu at (188.7, 95.7)
- added C279: 4.7uF, Capacitor_SMD:C_0603_1608Metric, F.Cu at (187.2, 96.2)
- added C283: 100nF, Capacitor_SMD:C_0402_1005Metric, F.Cu at (253.5, 84.2)
- added C286: 100nF, Capacitor_SMD:C_0402_1005Metric, B.Cu at (247.7, 47.0)
- added C288: 100nF, Capacitor_SMD:C_0402_1005Metric, B.Cu at (237.7, 49.7)
- added C309: 100nF, Capacitor_SMD:C_0402_1005Metric, B.Cu at (236.7, 49.6)
- added C318: 100nF, Capacitor_SMD:C_0402_1005Metric, B.Cu at (246.1, 43.6)
- added C319: 100nF, Capacitor_SMD:C_0402_1005Metric, B.Cu at (246.8, 42.9)
- added C320: 100nF, Capacitor_SMD:C_0402_1005Metric, B.Cu at (241.7, 37.6)
- added C321: 100nF, Capacitor_SMD:C_0402_1005Metric, B.Cu at (242.7, 37.6)
- added C322: tbd, Capacitor_SMD:C_1206_3216Metric, B.Cu at (258.2, 79.0)
- added C323: 100nF, Capacitor_SMD:C_0402_1005Metric, F.Cu at (180.1, 115.5)
- added D26: DF1501S-T, RASBB:DF1501ST, B.Cu at (243.5, 90.2)
- added D27: SMAJ33A, RASBB:DIOM5026X229N, F.Cu at (259.0, 102.5)
- added IC15: DS90LV028AQDQFRQ1, RASBB:SON50P200X200X80-8N, F.Cu at (247.0, 81.0)
- added J19: HC-WK88-H16-DB, RASBB:HC-WK88-H16-DB, F.Cu at (265.4, 89.2)
- added J20: Conn_01x02_Pin, Connector_PinHeader_2.54mm:PinHeader_1x02_P2.54mm_Vertical, F.Cu at (117.7, 107.2)
- added R186: 270, Resistor_SMD:R_0402_1005Metric, B.Cu at (259.1, 93.5)
- added R187: 100, Resistor_SMD:R_0402_1005Metric, F.Cu at (243.8, 81.8)
- added R188: 100, Resistor_SMD:R_0402_1005Metric, F.Cu at (243.8, 80.5)
- added R189: 100, Resistor_SMD:R_0402_1005Metric, F.Cu at (249.5, 82.2)
- added R190: 100, Resistor_SMD:R_0402_1005Metric, F.Cu at (249.5, 80.2)
- added R191: 10K, Resistor_SMD:R_0402_1005Metric, F.Cu at (251.5, 84.2)
- added R192: 10K, Resistor_SMD:R_0402_1005Metric, F.Cu at (251.5, 79.8)
- added R193: 10K, Resistor_SMD:R_0402_1005Metric, F.Cu at (251.5, 82.5)
- added R194: 10K, Resistor_SMD:R_0402_1005Metric, F.Cu at (251.5, 81.2)
- added R195: 10K, Resistor_SMD:R_0603_1608Metric, F.Cu at (126.2, 105.5)
- added R196: 4K7, Resistor_SMD:R_0402_1005Metric, B.Cu at (166.0, 114.8)
- added R197: 4K7, Resistor_SMD:R_0402_1005Metric, B.Cu at (167.2, 103.5)
- added R198: 4K7, Resistor_SMD:R_0402_1005Metric, B.Cu at (168.8, 63.4)
- added R199: 4K7, Resistor_SMD:R_0402_1005Metric, B.Cu at (169.2, 74.5)
- added R200: 10K, Resistor_SMD:R_0603_1608Metric, F.Cu at (193.2, 72.3)
- added R201: 10K, Resistor_SMD:R_0603_1608Metric, F.Cu at (193.2, 77.8)
- added R202: 10K, Resistor_SMD:R_0402_1005Metric, B.Cu at (259.1, 95.9)
- added R203: 2.49K, Resistor_SMD:R_0402_1005Metric, F.Cu at (204.3, 89.8)
- added R204: 4K7, Resistor_SMD:R_0402_1005Metric, F.Cu at (141.2, 53.0)
- added R205: 1.5K, Resistor_SMD:R_0402_1005Metric, F.Cu at (134.4, 53.0)
- added R206: 1.5K, Resistor_SMD:R_0402_1005Metric, F.Cu at (128.0, 102.8)
- added R207: 4K7, Resistor_SMD:R_0402_1005Metric, F.Cu at (119.0, 102.8)
- added R208: 0, Resistor_SMD:R_1206_3216Metric, F.Cu at (109.8, 111.3)
- added R209: 0, Resistor_SMD:R_1206_3216Metric, F.Cu at (107.0, 111.3)
- added R210: 270, Resistor_SMD:R_0402_1005Metric, F.Cu at (230.3, 74.8)
- added SW1: 435451019820, RASBB:435451019820, F.Cu at (188.6, 72.1)
- added SW2: 435451019820, RASBB:435451019820, F.Cu at (188.4, 77.7)
- added T1: 15FB-30NL, RASBB:SOIC127P940X597-16N, F.Cu at (247.0, 92.5)
- added TP24: TestPoint, TestPoint:TestPoint_Pad_D1.0mm, F.Cu at (174.7, 105.7)
- added TP25: TestPoint, TestPoint:TestPoint_Pad_D1.0mm, F.Cu at (187.2, 112.7)
- added U5: TLV9001DBVR, Package_TO_SOT_SMD:SOT-23-5, B.Cu at (122.0, 107.8)
- C139, C140: footprint Capacitor_SMD:C_0603_1608Metric -> Capacitor_SMD:C_0402_1005Metric
- C237: value 22uF -> 100nF; footprint Capacitor_SMD:C_0603_1608Metric -> Capacitor_SMD:C_0402_1005Metric
- C240: value 22uF -> 100nF; footprint Capacitor_SMD:C_0603_1608Metric -> Capacitor_SMD:C_0402_1005Metric; moved to B.Cu
- C256, D10, R83: moved to B.Cu
- IC10, IC9: value MT41K256M16TW-107_P -> MT41K128M16JT-107:K
- J14: value HR911196AE -> 636101112001; footprint RASBB:JK00229NL -> RASBB:J_Wurth_WR-UMRF_636101112001
- R150: value 270 -> 0; footprint Resistor_SMD:R_0402_1005Metric -> Resistor_SMD:R_0603_1608Metric; moved to F.Cu
- R151: value 270 -> 10K; footprint Resistor_SMD:R_0402_1005Metric -> Resistor_SMD:R_0603_1608Metric; moved to F.Cu
- R152, R153, R154, R155, R160, R161, R162, R163: value 100 -> 49.9
- R168, R169, R170, R171, R172, R173, R174, R175, R176, R177, R178, R179, R180, R181, R182, R183, R184: footprint Resistor_SMD:R_0201_0603Metric -> Resistor_SMD:R_0402_1005Metric
- R36: value 100K -> 220K
- moved C240 209.3 mm to (246.8, 47.9), turned to 135 degrees
- moved C237 206.6 mm to (245.8, 83.8)
- moved C256 117.2 mm to (156.7, 82.2), turned to 180 degrees
- moved C125 106.0 mm to (176.7, 82.3), turned to 180 degrees
- moved R150 105.4 mm to (120.7, 110.0), turned to -90 degrees
- moved R151 100.1 mm to (123.0, 105.5), turned to 0 degrees
- moved C181 31.4 mm to (233.8, 93.0), turned to -90 degrees
- moved R83 28.8 mm to (258.8, 81.5), turned to -90 degrees
- moved R144 22.1 mm to (234.8, 89.7), turned to 0 degrees
- moved R145 22.1 mm to (234.8, 87.8), turned to 0 degrees
- moved R143 22.1 mm to (231.7, 88.8), turned to 90 degrees
- moved D10 18.8 mm to (252.8, 89.8), turned to 0 degrees
- moved C183 14.7 mm to (258.5, 100.8), turned to -90 degrees
- moved C49 8.90 mm to (181.5, 57.8)
- moved C38 8.78 mm to (173.2, 57.8)
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Connections:
- C177 pad 1: /Ethernet_uC/RX_P -> /Ethernet_uC/RD_P
- C178 pad 1: /Ethernet_uC/RX_N -> /Ethernet_uC/RD_N
- C179 pad 1: /Ethernet_uC/TX_P -> /Ethernet_uC/TD_P
- C180 pad 1: /Ethernet_uC/TX_N -> /Ethernet_uC/TD_N
- C237 pad 1: GND -> +3V3
- C237 pad 2: +3V3 -> GND
- C240 pad 1: GND -> /FPGA-01/F1_B15_B18
- C240 pad 2: +3V3 -> /HDMI/HDMI_D2_P
- D10 pad 1: /Ethernet_uC/RX_P -> /Ethernet_uC/RD_P
- D10 pad 3: /Ethernet_uC/RX_N -> /Ethernet_uC/RD_N
- D10 pad 4: /Ethernet_uC/TX_P -> /Ethernet_uC/TD_P
- D10 pad 6: /Ethernet_uC/TX_N -> /Ethernet_uC/TD_N
- F2 pad 1: Net-(C16-Pad1) -> Net-(F2-Pad1)
- F2 pad 2: +12V -> Net-(C16-Pad1)
- IC12 pad 17: unconnected-(IC12-PC2_C-Pad17) -> /FPGA2_RESET
- IC12 pad 20: /FPGA-01/BANK0/FPGA1_DONE -> Net-(IC12-VREF+)
- IC12 pad 22: unconnected-(IC12-PA0-Pad22) -> /FPGA-01/BANK0/FPGA1_DONE
- IC12 pad 57: /uController/PD10_DEBUG -> Net-(IC12-PD10)
- IC12 pad 81: /uController/PD0_DEBUG -> Net-(IC12-PD0)
- IC12 pad 97: unconnected-(IC12-PE0-Pad97) -> /FPGA1_RESET
- IC14 pad 20: /Ethernet_uC/TX_N -> /Ethernet_uC/TD_N
- IC14 pad 21: /Ethernet_uC/TX_P -> /Ethernet_uC/TD_P
- IC14 pad 22: /Ethernet_uC/RX_N -> /Ethernet_uC/RD_N
- IC14 pad 23: /Ethernet_uC/RX_P -> /Ethernet_uC/RD_P
- IC5 pad 3: unconnected-(IC5-WP#/IO2-Pad3) -> Net-(IC5-WP#/IO2)
- IC5 pad 7: unconnected-(IC5-IO3/RESET#-Pad7) -> Net-(IC5-IO3/RESET#)
- IC7 pad 3: unconnected-(IC7-WP#/IO2-Pad3) -> Net-(IC7-WP#/IO2)
- IC7 pad 7: unconnected-(IC7-IO3/RESET#-Pad7) -> Net-(IC7-IO3/RESET#)
- J14 pad 1: unconnected-(J14-MDCT3-Pad1) -> Net-(J14-In)
- J14 pad 2: unconnected-(J14-MD3--Pad2) -> GND
- J4 pad A01: unconnected-(J4-PadA01) -> Net-(J4-PadA01)
- J4 pad A02: unconnected-(J4-PadA02) -> Net-(J4-PadA01)
- J4 pad A03: unconnected-(J4-PadA03) -> Net-(J4-PadA01)
- J4 pad B01: unconnected-(J4-PadB01) -> Net-(J4-PadA01)
- J4 pad B02: unconnected-(J4-PadB02) -> Net-(J4-PadA01)
- J4 pad B03: unconnected-(J4-PadB03) -> Net-(J4-PadA01)
- J8 pad 1: /uController/PD0_DEBUG -> +3V3
- J8 pad 10: /uController/PD10_DEBUG -> GND
- R139 pad 1: /Ethernet_uC/RX_P -> /Ethernet_uC/RD_P
- R140 pad 1: /Ethernet_uC/RX_N -> /Ethernet_uC/RD_N
- R141 pad 1: /Ethernet_uC/TX_P -> /Ethernet_uC/TD_P
- R142 pad 1: /Ethernet_uC/TX_N -> /Ethernet_uC/TD_N
- R144 pad 2: Net-(J14-MDCT1) -> Net-(R144-Pad2)
- R145 pad 2: Net-(J14-MDCT2) -> Net-(R145-Pad2)
- R150 pad 1: Net-(J14-GN_K) -> Net-(J20-Pin_2)
- R150 pad 2: GND -> Net-(U5--)
- R151 pad 1: Net-(J14-YL_K) -> Net-(U5-+)
- R151 pad 2: GND -> Net-(C272-Pad1)
- R83 pad 1: Net-(J2-YL_K) -> Net-(J19-Pad9)
- U10 pad A13: /HDMI/HDMI_CLK_P -> /FPGA-01/F1_B15_A13
- U10 pad A14: /HDMI/HDMI_CLK_N -> /FPGA-01/F1_B15_A14
- U10 pad A15: /HDMI/HDMI_D1_P -> /FPGA-01/F1_B15_A15
- U10 pad A16: /HDMI/HDMI_D1_N -> /FPGA-01/F1_B15_A16
- U10 pad A18: /HDMI/HDMI_D2_N -> /FPGA-01/F1_B15_A18
- U10 pad B16: /HDMI/HDMI_D0_P -> /FPGA-01/F1_B15_B16
- U10 pad B17: /HDMI/HDMI_D0_N -> /FPGA-01/F1_B15_B17
- U10 pad B18: /HDMI/HDMI_D2_P -> /FPGA-01/F1_B15_B18
- U10 pad F18: unconnected-(U10A-IO_L22N_T3_A16_15-PadF18) -> /FPGA1_RESET
- U10 pad G18: unconnected-(U10A-IO_L22P_T3_A17_15-PadG18) -> /CLK_OVR_ETH
- U10 pad U2: /DDR3-01/DDR301_UDQS_N -> /DDR3-01/DDR301_UDQS_P
- U10 pad V2: /DDR3-01/DDR301_UDQS_P -> /DDR3-01/DDR301_UDQS_N
- U11 pad C17: /FPGA-02/F2_B15_C17 -> /FPGA2_RESET
- U11 pad J2: unconnected-(U11C-IO_L22N_T3_35-PadJ2) -> /FPGA-02/F2_B35_J2
- U11 pad K13: /FPGA-02/F2_B15_K13 -> unconnected-(U11A-IO_L17P_T2_A26_15-PadK13)
- U11 pad K15: /FPGA-02/F2_B15_K15 -> unconnected-(U11A-IO_L24P_T3_RS1_15-PadK15)
- U11 pad L16: unconnected-(U11A-IO_L3N_T0_DQS_EMCCLK_14-PadL16) -> /CLK_OVR_ETH
- U12 pad 39: unconnected-(U12-RSET-Pad39) -> Net-(U12-RSET)
- U2 pad 2: /VSS_POE -> GND
- U2 pad 3: GND -> /VSS_POE
Routing:
- net +12V: track 15.1 -> 267.7 mm, vias 58 -> 59
- net +5V: track 282.2 -> 436.3 mm, vias 7 -> 8
- net /CLK_OVR_ETH: track 0.00 -> 152.1 mm, vias 0 -> 3
- net /FPGA-01/F1_B15_B16: track 0.00 -> 119.3 mm, vias 0 -> 2
- net /FPGA-01/F1_B15_B17: track 0.00 -> 119.3 mm, vias 0 -> 2
- net /FPGA-01/F1_B15_A14: track 0.00 -> 119.1 mm, vias 0 -> 2
- net /FPGA-01/F1_B15_A13: track 0.00 -> 117.2 mm, vias 0 -> 2
- net /HDMI/HDMI_D0_P: track 148.3 -> 31.2 mm, vias 2 -> 0
- net /HDMI/HDMI_D0_N: track 146.7 -> 29.7 mm, vias 2 -> 0
- net /HDMI/HDMI_CLK_N: track 136.3 -> 21.6 mm, vias 2 -> 0
- net /HDMI/HDMI_CLK_P: track 136.9 -> 22.6 mm, vias 2 -> 0
- net /FPGA-01/F1_B15_A18: track 0.00 -> 109.4 mm, vias 0 -> 2
- net /HDMI/HDMI_D2_N: track 163.3 -> 54.4 mm, vias 2 -> 0
- net /FPGA-01/F1_B15_B18: track 0.00 -> 107.3 mm, vias 0 -> 2
- net /HDMI/HDMI_D2_P: track 156.3 -> 49.4 mm, vias 2 -> 0
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Other:
- board text added: "DNP R208 IF R209 IS POPULATED"
- board text added: "RASBB Rev. C"
- board text removed: "MD Design 2025"
- board text removed: "RASBB Rev. B"
