File: RASBB/Hardware/Rev.C/Design/Audio_IN-OUT.kicad_sch (KiCad schematic)
At the start: 20 parts, among them J12 AudioJack4, U8 LM386, U9 LM321

Commit message: Draft AC
Parts:
- J12: LCSC Order # C7501803 -> (none)
- R127: LCSC Part # C163810 -> C168239; Mfr. Part # WR04X1002FTL -> WR04X5601FTL
- U9: Mfr. Part # (none) -> LM321-TR
Changed lines of the file:
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@@
 			)
 		)
-		(property "Description" "62.5mW Thick Film Resistors 50V ±100ppm/℃ ±1% 10kΩ 0402 Chip Resistor - Surface Mount ROHS"
+		(property "Description" "Resistor, small symbol"
 			(at 193.04 95.25 0)
 			(hide yes)
@@
 			)
 		)
-		(property "Description" "62.5mW Thick Film Resistors 50V ±100ppm/℃ ±1% 1.2kΩ 0402 Chip Resistor - Surface Mount ROHS"
+		(property "Description" "Resistor, small symbol"
 			(at 93.98 60.96 0)
 			(hide yes)
@@
 			)
 		)
-		(property "Description" "62.5mW Thick Film Resistors 50V ±100ppm/℃ ±1% 100kΩ 0402 Chip Resistor - Surface Mount ROHS"
+		(property "Description" "Resistor, small symbol"
 			(at 157.48 123.19 0)
 			(hide yes)
@@
 			)
 		)
+		(property "Mfr. Part #" "LM321-TR"
+			(at 121.92 113.03 0)
+			(hide yes)
+			(show_name no)
+			(do_not_autoplace no)
+			(effects
+				(font
+					(size 1.27 1.27)
+				)
+			)
+		)
 		(pin "4"
 		)
@@
 			)
 		)
-		(property "Datasheet" "https://www.lcsc.com/datasheet/lcsc_datasheet_2309201533_Walsin-Tech-Corp-0402B103K100CT_C3840241.pdf"
+		(property "Datasheet" ""
 			(at 76.2 26.67 0)
 			(hide yes)
@@
 			)
 		)
-		(property "Description" "10V 100nF X7R ±10% 0402 Multilayer Ceramic Capacitors MLCC - SMD/SMT ROHS"
+		(property "Description" "50V 100nF X7R ±10% 0402 Multilayer Ceramic Capacitors MLCC - SMD/SMT ROHS"
 			(at 76.2 26.67 0)
 			(hide yes)
@@
 			)
 		)
-		(property "Datasheet" "https://www.lcsc.com/datasheet/lcsc_datasheet_2309201533_Walsin-Tech-Corp-0402B103K100CT_C3840241.pdf"
+		(property "Datasheet" ""
 			(at 124.46 123.19 0)
 			(hide yes)
@@
 			)
 		)
-		(property "Description" "10V 100nF X7R ±10% 0402 Multilayer Ceramic Capacitors MLCC - SMD/SMT ROHS"
+		(property "Description" "50V 100nF X7R ±10% 0402 Multilayer Ceramic Capacitors MLCC - SMD/SMT ROHS"
 			(at 124.46 123.19 0)
 			(hide yes)
@@
 			)
 		)
-		(property "Datasheet" "https://www.lcsc.com/datasheet/lcsc_datasheet_2304140030_Samsung-Electro-Mechanics-CL05A105KP5NNNC_C14445.pdf"
+		(property "Datasheet" ""
 			(at 168.91 115.57 0)
 			(hide yes)
@@
 			)
 		)
-		(property "Description" "10V 1uF X5R ±10% 0402 Multilayer Ceramic Capacitors MLCC - SMD/SMT ROHS"
+		(property "Description" "16V 1uF X5R ±20% 0402 Multilayer Ceramic Capacitors MLCC - SMD/SMT ROHS"
 			(at 168.91 115.57 0)
 			(hide yes)
@@
 			)
 		)
-		(property "Datasheet" "https://www.lcsc.com/datasheet/lcsc_datasheet_2304140030_Walsin-Tech-Corp-0402B473K250CT_C314287.pdf"
+		(property "Datasheet" ""
 			(at 114.3 50.8 0)
 			(hide yes)
@@
 			)
 		)
-		(property "Description" "25V 47nF X7R ±10% 0402 Multilayer Ceramic Capacitors MLCC - SMD/SMT ROHS"
+		(property "Description" "10V 47nF X7R ±5% 0402 Multilayer Ceramic Capacitors MLCC - SMD/SMT ROHS"
 			(at 114.3 50.8 0)
 			(hide yes)
@@
 			)
 		)
-		(property "Description" "62.5mW Thick Film Resistors 50V ±100ppm/℃ ±1% 10kΩ 0402 Chip Resistor - Surface Mount ROHS"
+		(property "Description" "Resistor, small symbol"
 			(at 134.62 138.43 0)
 			(hide yes)
@@
 			)
 		)
-		(property "LCSC Order #" "C7501803"
+		(property "LCSC Order #" ""
 			(at 227.584 121.412 0)
 			(hide yes)
@@
 			)
 		)
-		(property "Description" "62.5mW Thick Film Resistors 50V ±1% ±200ppm/℃ 10Ω 0402 Chip Resistor - Surface Mount ROHS"
+		(property "Description" "Resistor, small symbol"
 			(at 114.3 43.18 0)
 			(hide yes)
@@
 			)
 		)
-		(property "Datasheet" "https://www.lcsc.com/datasheet/lcsc_datasheet_2304140030_Walsin-Tech-Corp-WR04X1002FTL_C163810.pdf"
+		(property "Datasheet" ""
 			(at 181.61 110.49 0)
 			(hide yes)
@@
 			)
 		)
-		(property "Description" "62.5mW Thick Film Resistors 50V ±100ppm/℃ ±1% 10kΩ 0402 Chip Resistor - Surface Mount ROHS"
+		(property "Description" "Resistor, small symbol"
 			(at 181.61 110.49 0)
 			(hide yes)
@@
 			)
 		)
-		(property "Mfr. Part #" "WR04X1002FTL "
+		(property "Mfr. Part #" "WR04X5601FTL"
 			(at 181.61 110.49 0)
 			(hide yes)
@@
 			)
 		)
-		(property "LCSC Part #" "C163810"
+		(property "LCSC Part #" "C168239"
 			(at 181.61 110.49 0)
 			(hide yes)
@@
 			)
 		)
-		(property "Description" "62.5mW Thick Film Resistors 50V ±100ppm/℃ ±1% 100kΩ 0402 Chip Resistor - Surface Mount ROHS"
+		(property "Description" "Resistor, small symbol"
 			(at 157.48 109.22 0)
 			(hide yes)

Commit message: Modified Based on Findings -Draft
Parts:
- R125, R126: now fitted
Changed lines of the file:
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@@
 	(title_block
 		(title "RASBB")
-		(date "2026-07-25")
+		(date "2026-09-20")
 		(rev "C")
 		(company "Mina Daneshpajouh")
@@
 		(on_board yes)
 		(in_pos_files yes)
-		(dnp yes)
+		(dnp no)
 		(property "Reference" "R126"
 			(at 154.686 122.682 90)
@@
 		(on_board yes)
 		(in_pos_files yes)
-		(dnp yes)
+		(dnp no)
 		(property "Reference" "R125"
 			(at 160.02 109.474 90)
