File: RASBB/Hardware/Rev.C/Design/Ethernet_FPGA.kicad_sch (KiCad schematic)
At the start: 52 parts, among them J2 HR911196AE, J6 HC-WK88-H16-DB, U12 RTL8211E-VB-CG, X1 OT2EL4C4JI-111OLP-50M

Commit message: Draft AC
Parts:
- removed J6: HC-WK88-H16-DB, symbol RASBB_Library:HC-WK88-H16-DB
- added R203: 2.49K, Resistor_SMD:R_0402_1005Metric, symbol Device:R
- added R210: 270, Resistor_SMD:R_0402_1005Metric, symbol Device:R
- J2: Mfr. Part # (none) -> HR911196AE
- R107, R57, R58, R59, R60, R61, R62, R74, R76: LCSC Part #  C163826 -> (none)
- U12: LCSC Part #  C90735 -> (none)
- X1: Mfr. Part # (none) -> OT2EL4C4JI-111OLP-50M
Connections:
- net GND: now also R203.2, R210.2
- net LED_YL_ETH: now also J2.19 (YL_A)
- net at U12.39 (RSET): now also R203.1
- net at J2.20 (YL_K): now also R210.1
