File: RASBB/Hardware/Rev.C/Design/Ethernet_uC.kicad_sch (KiCad schematic)
At the start: 59 parts, among them IC14 LAN8742AI-CZ-TR, IC15 DS90LV028AQDQFRQ1, J14 636101112001, J19 HC-WK88-H16-DB, T1 15FB-30NL, Y3 25MHz

Commit message: Draft AC
Parts:
- removed C240: 100nF, Capacitor_SMD:C_0402_1005Metric, symbol Device:C_Small
- added C283: 100nF, Capacitor_SMD:C_0402_1005Metric, symbol Device:C_Small
- added C322: tbd, Capacitor_SMD:C_1206_3216Metric, symbol Device:C_Small
- added R202: 10K, Resistor_SMD:R_0402_1005Metric, symbol Device:R_Small
- C126: LCSC Part # C3840241 -> C301927; Mfr. Part # 0402B103K100CT -> 0402B103K500CT
- C168, C176: LCSC Part # C2178655 -> C301961; Mfr. Part # (none) -> 0402N100J500CT
- C175: LCSC Part # C913474 -> C7281848; Mfr. Part # GRM188Z71A475KE15D -> GMK107BBJ475KA-T
- C177, C178, C179, C180: LCSC Part # C123155 -> C152928; Mfr. Part # (none) -> 0603N100J500CT
- C66: Mfr. Part # C526993 -> CC0402JRNPO7BN471
- IC15: footprint SON50P200X200X80-8N -> RASBB:SON50P200X200X80-8N; LCSC Part # (none) -> C2868409; Mfr. Part # (none) -> DS90LV028AQDQFRQ1
- J14: footprint Connector_SMD_Wurth:J_Wurth_WR-UMRF_636101112001 -> RASBB:J_Wurth_WR-UMRF_636101112001; Mfr. Part # (none) -> 636101112001
- J19: LCSC Part # (none) -> C7501824; Mfr. Part # (none) -> HC-WK88-H16-DB
- R187, R188, R189, R190: footprint Resistor_SMD:R_0201_0603Metric -> Resistor_SMD:R_0402_1005Metric; LCSC Part # C367410 -> C163808; Mfr. Part # WR02X1000FTL -> WR04X1000FTL
- T1: LCSC Part # (none) -> C2987675; Mfr. Part # (none) -> 15FB-30NL
- Y3: Mfr. Part # (none) -> XL2EL89CSI-111YLC-25M
Connections:
- net GND: now also C322.2, R202.2
- net LED_YL_ETH: now also R202.1
- net at C268.1, IC15.4 (RIN2-), R194.1: now also R190.2; no longer R190.1
- net at IC15.1 (RIN1-), R191.2: now also R189.1, C283.1; no longer R189.2
- net at C259.1, IC15.2 (RIN1+): now also R189.2, R193.1; no longer R189.1
- net at C260.1, IC15.3 (RIN2+): now also R190.1, R192.2; no longer R190.2
- net at C183.1, J19.S1, J19.S2: now also C322.1
- net CLK_OVR_ETH: now reaches R187.2
- removed net +: C259.2, C260.2, J19.5, J19.7, R192.2, R193.1
- net ++ renamed RIN2_N
- net RIN2_N: now also J19.5; no longer J19.4
- net - renamed RIN1_N
- net RIN1_N: now also C283.2
- net RX_N renamed RD_N
- net RD_N: no longer J19.6, T1.9 (RX-)
- net RX_P renamed RD_P
- net RD_P: no longer J19.3, T1.11 (RX+)
- net TX_N renamed TD_N
- net TD_N: no longer J19.2, T1.14 (TX-)
- net TX_P renamed TD_P
- net TD_P: no longer J19.1, T1.16 (TX+)
- new net ETH_RX_N: J19.6, T1.9 (RX-)
- new net ETH_RX_P: J19.3, T1.11 (RX+)
- new net ETH_TX_N: J19.2, T1.14 (TX-)
- new net ETH_TX_P: J19.1, T1.16 (TX+)
- new net RIN1_P: C259.2, J19.7
- new net RIN2_P: C260.2, J19.4
Other:
- note removed: "To FPGA 1/2"
- note removed: "To SMA connector"
- moved on the sheet: C126, C183, C237, C259, IC15, J14, J19, R186, R187, R191, R192, R194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
