File: RASBB/Hardware/Rev.C/Design/FPGA01.kicad_sch (KiCad schematic)
At the start: 0 parts

Commit message: Draft AC
Other:
- sheet BANK14-15 ports: added F1_B15_F18, F1_B15_G18; removed none
- sheet BANK16-34 ports: added DDR301_UDQS_P; removed DDR301_UQDS_P
Changed lines of the file:
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@@
 	(wire
 		(pts
+			(xy 462.28 184.15) (xy 477.52 184.15)
+		)
+		(stroke
+			(width 0)
+			(type default)
+		)
+	)
+	(wire
+		(pts
 			(xy 41.91 190.5) (xy 49.53 190.5)
 		)
@@
 	(wire
 		(pts
+			(xy 462.28 187.96) (xy 477.52 187.96)
+		)
+		(stroke
+			(width 0)
+			(type default)
+		)
+	)
+	(wire
+		(pts
 			(xy 176.53 166.37) (xy 186.69 166.37)
 		)
@@
 		)
 	)
+	(hierarchical_label "F1_B15_F18"
+		(shape input)
+		(at 462.28 184.15 180)
+		(effects
+			(font
+				(size 1.27 1.27)
+			)
+			(justify right)
+		)
+	)
 	(hierarchical_label "DDR301_BA2"
 		(shape output)
@@
 	)
 	(hierarchical_label "F1_B15_E18"
-		(shape output)
+		(shape input)
 		(at 466.09 139.7 180)
 		(effects
@@
 		)
 	)
+	(hierarchical_label "F1_B15_G18"
+		(shape input)
+		(at 462.28 187.96 180)
+		(effects
+			(font
+				(size 1.27 1.27)
+			)
+			(justify right)
+		)
+	)
 	(hierarchical_label "F1_B14_U17"
 		(shape bidirectional)
@@
 		)
 	)
-	(hierarchical_label "DDR301_UDQS_P"
+	(hierarchical_label "DDR301_UDQS_N"
 		(shape output)
 		(at 377.19 186.69 0)
@@
 		)
 	)
-	(hierarchical_label "DDR301_UDQS_N"
+	(hierarchical_label "DDR301_UDQS_P"
 		(shape output)
 		(at 377.19 184.15 0)
@@
 			)
 		)
+		(pin "F1_B15_F18" input
+			(at 477.52 184.15 180)
+			(effects
+				(font
+					(size 1.27 1.27)
+				)
+				(justify left)
+			)
+		)
+		(pin "F1_B15_G18" input
+			(at 477.52 187.96 180)
+			(effects
+				(font
+					(size 1.27 1.27)
+				)
+				(justify left)
+			)
+		)
 		(instances
 			(project "RASBB"
@@
 			)
 		)
-		(pin "DDR301_UQDS_P" output
-			(at 369.57 184.15 0)
-			(effects
-				(font
-					(size 1.27 1.27)
-				)
-				(justify right)
-			)
-		)
 		(pin "DDR301_DQ14" bidirectional
 			(at 369.57 158.75 0)
@@
 			(effects
 				(font
+					(size 1.27 1.27)
+				)
+				(justify right)
+			)
+		)
+		(pin "DDR301_UDQS_P" output
+			(at 369.57 184.15 0)
+			(effects
+				(font
