File: RASBB/Hardware/Rev.C/Design/FPGA02.kicad_sch (KiCad schematic)
At the start: 0 parts

Commit message: Draft AC
Other:
- sheet BANK14-15 ports: added FPGA2_B14_L16; removed F2_B15_K13, F2_B15_K15
- sheet BANK35 ports: added F2_B35_J2; removed none
Changed lines of the file:
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@@
 	(wire
 		(pts
-			(xy 471.17 220.98) (xy 482.6 220.98)
-		)
-		(stroke
-			(width 0)
-			(type default)
-		)
-	)
-	(wire
-		(pts
 			(xy 471.17 200.66) (xy 482.6 200.66)
 		)
@@
 	(wire
 		(pts
-			(xy 471.17 223.52) (xy 482.6 223.52)
-		)
-		(stroke
-			(width 0)
-			(type default)
-		)
-	)
-	(wire
-		(pts
 			(xy 374.65 160.02) (xy 382.27 160.02)
 		)
@@
 	(wire
 		(pts
+			(xy 181.61 217.17) (xy 191.77 217.17)
+		)
+		(stroke
+			(width 0)
+			(type default)
+		)
+	)
+	(wire
+		(pts
 			(xy 374.65 170.18) (xy 382.27 170.18)
 		)
@@
 	(wire
 		(pts
+			(xy 543.56 173.99) (xy 524.51 173.99)
+		)
+		(stroke
+			(width 0)
+			(type default)
+		)
+	)
+	(wire
+		(pts
 			(xy 471.17 177.8) (xy 482.6 177.8)
 		)
@@
 		)
 	)
-	(hierarchical_label "F2_B15_K13"
-		(shape bidirectional)
-		(at 471.17 220.98 180)
-		(effects
-			(font
-				(size 1.27 1.27)
-			)
-			(justify right)
-		)
-	)
 	(hierarchical_label "F2_B15_E18"
 		(shape bidirectional)
@@
 	)
 	(hierarchical_label "F2_B15_C17"
-		(shape bidirectional)
+		(shape input)
 		(at 471.17 152.4 180)
 		(effects
@@
 		)
 	)
-	(hierarchical_label "F2_B15_K15"
-		(shape bidirectional)
-		(at 471.17 223.52 180)
-		(effects
-			(font
-				(size 1.27 1.27)
-			)
-			(justify right)
-		)
-	)
 	(hierarchical_label "F2_B34_L6"
 		(shape bidirectional)
@@
 		)
 	)
+	(hierarchical_label "F2_B35_J2"
+		(shape output)
+		(at 181.61 217.17 180)
+		(effects
+			(font
+				(size 1.27 1.27)
+				(thickness 0.254)
+				(bold yes)
+			)
+			(justify right)
+		)
+	)
 	(hierarchical_label "F2_B34_T3"
 		(shape bidirectional)
@@
 		)
 	)
+	(hierarchical_label "F2_B14_L16"
+		(shape output)
+		(at 543.56 173.99 0)
+		(effects
+			(font
+				(size 1.27 1.27)
+			)
+			(justify left)
+		)
+	)
 	(hierarchical_label "F2_B34_N1"
 		(shape output)
@@
 			)
 		)
-		(pin "F2_B35_E1" input
+		(pin "F2_B35_E1" output
 			(at 191.77 213.36 180)
 			(effects
@@
 			)
 		)
+		(pin "F2_B35_J2" output
+			(at 191.77 217.17 180)
+			(effects
+				(font
+					(size 1.27 1.27)
+				)
+				(justify left)
+			)
+		)
 		(instances
 			(project "RASBB"
@@
 			)
 		)
-		(pin "F2_B15_C17" bidirectional
+		(pin "F2_B15_C17" input
 			(at 482.6 152.4 180)
 			(effects
@@
 			)
 		)
-		(pin "F2_B15_K13" bidirectional
-			(at 482.6 220.98 180)
-			(effects
-				(font
-					(size 1.27 1.27)
-				)
-				(justify left)
-			)
-		)
-		(pin "F2_B15_K15" bidirectional
-			(at 482.6 223.52 180)
-			(effects
-				(font
-					(size 1.27 1.27)
-				)
-				(justify left)
-			)
-		)
 		(pin "F2_B15_K16" bidirectional
 			(at 482.6 226.06 180)
@@
 			)
 		)
+		(pin "FPGA2_B14_L16" output
+			(at 524.51 173.99 0)
+			(effects
+				(font
+					(size 1.27 1.27)
+				)
+				(justify right)
+			)
+		)
