File: RASBB/Hardware/Rev.C/Design/FPGA1_BANK14-15.kicad_sch (KiCad schematic)
At the start: 27 parts, among them U10 XC7A100T-CSG324

Commit message: Draft AC
Connections:
- net F1_B15_F18: now reaches U10.F18 (IO_L22N_T3_A16_15)
- net F1_B15_G18: now reaches U10.G18 (IO_L22P_T3_A17_15)
- no-connect marks 0 -> 37
