File: RASBB/Hardware/Rev.C/Design/FPGA1_BANK16-34.kicad_sch (KiCad schematic)
At the start: 11 parts, among them U10 XC7A100T-CSG324

Commit message: Draft AC
Parts:
- C228: Mfr. Part # GRM155R61A475KEAAD -> GRM155R61A475KEAAD
Connections:
- net DDR301_UQDS_P renamed DDR301_UDQS_P
- no-connect marks 0 -> 11
Changed lines of the file:
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@@
 		(color 0 0 0 0)
 	)
+	(no_connect
+		(at 128.27 96.52)
+	)
+	(no_connect
+		(at 128.27 93.98)
+	)
+	(no_connect
+		(at 128.27 99.06)
+	)
+	(no_connect
+		(at 128.27 86.36)
+	)
+	(no_connect
+		(at 128.27 81.28)
+	)
+	(no_connect
+		(at 128.27 78.74)
+	)
+	(no_connect
+		(at 128.27 101.6)
+	)
+	(no_connect
+		(at 128.27 83.82)
+	)
+	(no_connect
+		(at 229.87 109.22)
+	)
+	(no_connect
+		(at 128.27 91.44)
+	)
+	(no_connect
+		(at 128.27 88.9)
+	)
 	(wire
 		(pts
@@
 	(wire
 		(pts
-			(xy 229.87 137.16) (xy 243.84 137.16)
+			(xy 229.87 195.58) (xy 243.84 195.58)
 		)
 		(stroke
@@
 	(wire
 		(pts
-			(xy 229.87 195.58) (xy 243.84 195.58)
+			(xy 229.87 187.96) (xy 243.84 187.96)
 		)
 		(stroke
@@
 	(wire
 		(pts
-			(xy 229.87 187.96) (xy 243.84 187.96)
+			(xy 229.87 167.64) (xy 243.84 167.64)
 		)
 		(stroke
@@
 	(wire
 		(pts
-			(xy 229.87 167.64) (xy 243.84 167.64)
+			(xy 229.87 137.16) (xy 243.84 137.16)
 		)
 		(stroke
@@
 	(wire
 		(pts
-			(xy 229.87 78.74) (xy 243.84 78.74)
-		)
-		(stroke
-			(width 0)
-			(type default)
-		)
-	)
-	(wire
-		(pts
 			(xy 229.87 86.36) (xy 243.84 86.36)
 		)
@@
 	(wire
 		(pts
+			(xy 229.87 78.74) (xy 243.84 78.74)
+		)
+		(stroke
+			(width 0)
+			(type default)
+		)
+	)
+	(wire
+		(pts
 			(xy 279.4 64.77) (xy 279.4 66.04)
 		)
@@
 		)
 	)
-	(hierarchical_label "DDR301_LDM"
+	(hierarchical_label "DDR301_A14"
 		(shape output)
-		(at 243.84 81.28 0)
-		(effects
-			(font
-				(size 1.27 1.27)
-			)
-			(justify left)
-		)
-	)
-	(hierarchical_label "DDR301_UQDS_P"
-		(shape bidirectional)
-		(at 243.84 121.92 0)
+		(at 243.84 137.16 0)
 		(effects
 			(font
@@
 		)
 	)
-	(hierarchical_label "DDR301_nCS"
+	(hierarchical_label "DDR301_LDM"
 		(shape output)
-		(at 243.84 203.2 0)
+		(at 243.84 81.28 0)
 		(effects
 			(font
@@
 		)
 	)
-	(hierarchical_label "DDR301_nCAS"
+	(hierarchical_label "DDR301_UDQS_P"
 		(shape output)
-		(at 243.84 157.48 0)
+		(at 243.84 121.92 0)
 		(effects
 			(font
@@
 		)
 	)
-	(hierarchical_label "DDR301_LDQS_N"
+	(hierarchical_label "DDR301_nCS"
 		(shape output)
-		(at 243.84 93.98 0)
+		(at 243.84 203.2 0)
 		(effects
 			(font
@@
 		)
 	)
-	(hierarchical_label "DDR301_nRST"
+	(hierarchical_label "DDR301_nCAS"
 		(shape output)
-		(at 243.84 78.74 0)
+		(at 243.84 157.48 0)
 		(effects
 			(font
@@
 		)
 	)
-	(hierarchical_label "DDR301_A14"
+	(hierarchical_label "DDR301_LDQS_N"
 		(shape output)
-		(at 243.84 137.16 0)
+		(at 243.84 93.98 0)
 		(effects
 			(font
@@
 		)
 	)
+	(hierarchical_label "DDR301_nRST"
+		(shape output)
+		(at 243.84 78.74 0)
+		(effects
+			(font
+				(size 1.27 1.27)
+			)
+			(justify left)
+		)
+	)
 	(hierarchical_label "DDR301_A11"
 		(shape output)
@@
 			)
 		)
-		(property "Datasheet" "https://www.lcsc.com/datasheet/lcsc_datasheet_2206281830_Murata-Electronics-GRT155R71A474KE01D_C711087.pdf"
+		(property "Datasheet" ""
 			(at 260.35 62.23 0)
 			(hide yes)
@@
 			)
 		)
-		(property "Description" "Unpolarized capacitor, small symbol"
+		(property "Description" "16V 470nF X7R ±10% 0402 Multilayer Ceramic Capacitors MLCC - SMD/SMT ROHS"
 			(at 260.35 62.23 0)
 			(hide yes)
@@
 			)
 		)
-		(property "Datasheet" "https://www.lcsc.com/datasheet/lcsc_datasheet_2206281830_Murata-Electronics-GRT155R71A474KE01D_C711087.pdf"
+		(property "Datasheet" ""
 			(at 270.51 62.23 0)
 			(hide yes)
@@
 			)
 		)
-		(property "Description" "Unpolarized capacitor, small symbol"
+		(property "Description" "16V 470nF X7R ±10% 0402 Multilayer Ceramic Capacitors MLCC - SMD/SMT ROHS"
 			(at 270.51 62.23 0)
 			(hide yes)
@@
 			)
 		)
-		(property "Datasheet" "https://www.lcsc.com/datasheet/lcsc_datasheet_2206281830_Murata-Electronics-GRT155R71A474KE01D_C711087.pdf"
+		(property "Datasheet" ""
 			(at 83.82 62.23 0)
 			(hide yes)
@@
 			)
 		)
-		(property "Description" "Unpolarized capacitor, small symbol"
+		(property "Description" "16V 470nF X7R ±10% 0402 Multilayer Ceramic Capacitors MLCC - SMD/SMT ROHS"
 			(at 83.82 62.23 0)
 			(hide yes)
@@
 			)
 		)
-		(property "Datasheet" "https://www.lcsc.com/datasheet/lcsc_datasheet_2206281830_Murata-Electronics-GRT155R71A474KE01D_C711087.pdf"
+		(property "Datasheet" ""
 			(at 279.4 62.23 0)
 			(hide yes)
@@
 			)
 		)
-		(property "Description" "Unpolarized capacitor, small symbol"
+		(property "Description" "16V 470nF X7R ±10% 0402 Multilayer Ceramic Capacitors MLCC - SMD/SMT ROHS"
 			(at 279.4 62.23 0)
 			(hide yes)
@@
 			)
 		)
-		(property "Datasheet" "https://www.lcsc.com/datasheet/lcsc_datasheet_1811081617_Murata-Electronics-GRM155R61A475KEAAD_C77004.pdf"
+		(property "Datasheet" ""
 			(at 241.3 62.23 0)
 			(hide yes)
@@
 			)
 		)
-		(property "Datasheet" "https://www.lcsc.com/datasheet/lcsc_datasheet_2201131300_Murata-Electronics-GRM188Z71A475KE15D_C913474.pdf"
+		(property "Datasheet" ""
 			(at 251.46 62.23 0)
 			(hide yes)
@@
 			)
 		)
-		(property "Mfr. Part #" "GRM155R61A475KEAAD"
+		(property "Mfr. Part #" "GRM155R61A475KEAAD "
 			(at 251.46 62.23 0)
 			(hide yes)
@@
 			)
 		)
-		(property "Datasheet" "https://www.lcsc.com/datasheet/lcsc_datasheet_1811081617_Murata-Electronics-GRM155R61A475KEAAD_C77004.pdf"
+		(property "Datasheet" ""
 			(at 74.93 62.23 0)
 			(hide yes)
@@
 			)
 		)
-		(property "Datasheet" "https://www.lcsc.com/datasheet/lcsc_datasheet_2206281830_Murata-Electronics-GRT155R71A474KE01D_C711087.pdf"
+		(property "Datasheet" ""
 			(at 287.02 62.23 0)
 			(hide yes)
@@
 			)
 		)
-		(property "Description" "Unpolarized capacitor, small symbol"
+		(property "Description" "16V 470nF X7R ±10% 0402 Multilayer Ceramic Capacitors MLCC - SMD/SMT ROHS"
 			(at 287.02 62.23 0)
 			(hide yes)
@@
 			)
 		)
-		(property "Datasheet" "https://www.lcsc.com/datasheet/lcsc_datasheet_2206281830_Murata-Electronics-GRT155R71A474KE01D_C711087.pdf"
+		(property "Datasheet" ""
 			(at 298.45 62.23 0)
 			(hide yes)
@@
 			)
 		)
-		(property "Description" "Unpolarized capacitor, small symbol"
+		(property "Description" "16V 470nF X7R ±10% 0402 Multilayer Ceramic Capacitors MLCC - SMD/SMT ROHS"
 			(at 298.45 62.23 0)
 			(hide yes)
@@
 			)
 		)
-		(property "Datasheet" "https://www.lcsc.com/datasheet/lcsc_datasheet_2201131300_Murata-Electronics-GRM188Z71A475KE15D_C913474.pdf"
+		(property "Datasheet" ""
 			(at 231.14 62.23 0)
 			(hide yes)
