File: RASBB/Hardware/Rev.C/Design/FPGA1_BANK35.kicad_sch (KiCad schematic)
At the start: 17 parts, among them J16 Conn_01x02_Pin, U10 XC7A100T-CSG324, X3 OT2EL4C4JI-111OLP-50M

Commit message: Draft AC
Parts:
- J16: LCSC Part # (none) -> C492401; Mfr. Part # (none) -> PZ254V-11-02P
- X3: Mfr. Part # (none) -> OT2EL4C4JI-111OLP-50M
Connections:
- no-connect marks 0 -> 14
Changed lines of the file:
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@@
 		(color 0 0 0 0)
 	)
+	(no_connect
+		(at 163.83 149.86)
+	)
+	(no_connect
+		(at 163.83 109.22)
+	)
+	(no_connect
+		(at 163.83 177.8)
+	)
+	(no_connect
+		(at 163.83 99.06)
+	)
+	(no_connect
+		(at 163.83 111.76)
+	)
+	(no_connect
+		(at 163.83 205.74)
+	)
+	(no_connect
+		(at 163.83 81.28)
+	)
+	(no_connect
+		(at 163.83 200.66)
+	)
+	(no_connect
+		(at 163.83 175.26)
+	)
+	(no_connect
+		(at 163.83 152.4)
+	)
+	(no_connect
+		(at 163.83 185.42)
+	)
+	(no_connect
+		(at 163.83 203.2)
+	)
+	(no_connect
+		(at 163.83 187.96)
+	)
+	(no_connect
+		(at 163.83 101.6)
+	)
 	(wire
 		(pts
@@
 			)
 		)
-		(property "Datasheet" "https://www.lcsc.com/datasheet/lcsc_datasheet_2206281830_Murata-Electronics-GRT155R71A474KE01D_C711087.pdf"
+		(property "Datasheet" ""
 			(at 144.78 64.77 0)
 			(hide yes)
@@
 			)
 		)
-		(property "Description" "10V 470nF X7R ±10% 0402 Multilayer Ceramic Capacitors MLCC - SMD/SMT ROHS"
+		(property "Description" "16V 470nF X7R ±10% 0402 Multilayer Ceramic Capacitors MLCC - SMD/SMT ROHS"
 			(at 144.78 64.77 0)
 			(hide yes)
@@
 			)
 		)
-		(property "Description" "62.5mW Thick Film Resistors ±100ppm/℃ ±1% 49.9Ω 0402 Chip Resistor - Surface Mount ROHS"
+		(property "Description" "Resistor, small symbol"
 			(at 123.19 142.24 0)
 			(hide yes)
@@
 			)
 		)
-		(property "Datasheet" "https://www.lcsc.com/datasheet/lcsc_datasheet_2206281830_Murata-Electronics-GRT155R71A474KE01D_C711087.pdf"
+		(property "Datasheet" ""
 			(at 134.62 64.77 0)
 			(hide yes)
@@
 			)
 		)
-		(property "Description" "10V 470nF X7R ±10% 0402 Multilayer Ceramic Capacitors MLCC - SMD/SMT ROHS"
+		(property "Description" "16V 470nF X7R ±10% 0402 Multilayer Ceramic Capacitors MLCC - SMD/SMT ROHS"
 			(at 134.62 64.77 0)
 			(hide yes)
@@
 			)
 		)
-		(property "Description" "62.5mW Thick Film Resistors ±100ppm/℃ ±1% 49.9Ω 0402 Chip Resistor - Surface Mount ROHS"
+		(property "Description" "Resistor, small symbol"
 			(at 96.52 139.7 0)
 			(hide yes)
@@
 			)
 		)
-		(property "Datasheet" "https://www.lcsc.com/datasheet/lcsc_datasheet_2206281830_Murata-Electronics-GRT155R71A474KE01D_C711087.pdf"
+		(property "Datasheet" ""
 			(at 106.68 64.77 0)
 			(hide yes)
@@
 			)
 		)
-		(property "Description" "10V 47nF X7R ±5% 0402 Multilayer Ceramic Capacitors MLCC - SMD/SMT ROHS"
+		(property "Description" "16V 470nF X7R ±10% 0402 Multilayer Ceramic Capacitors MLCC - SMD/SMT ROHS"
 			(at 106.68 64.77 0)
 			(hide yes)
@@
 			)
 		)
-		(property "Description" "62.5mW Thick Film Resistors ±100ppm/℃ ±1% 49.9Ω 0402 Chip Resistor - Surface Mount ROHS"
+		(property "Description" "Resistor, small symbol"
 			(at 87.63 130.81 0)
 			(hide yes)
@@
 			)
 		)
+		(property "Mfr. Part #" "OT2EL4C4JI-111OLP-50M"
+			(at 58.42 139.7 0)
+			(hide yes)
+			(show_name no)
+			(do_not_autoplace no)
+			(effects
+				(font
+					(size 1.27 1.27)
+				)
+			)
+		)
 		(pin "4"
 		)
@@
 			)
 		)
-		(property "Datasheet" "https://www.lcsc.com/datasheet/lcsc_datasheet_2206281830_Murata-Electronics-GRT155R71A474KE01D_C711087.pdf"
+		(property "Datasheet" ""
 			(at 118.11 64.77 0)
 			(hide yes)
@@
 			)
 		)
-		(property "Description" "10V 470nF X7R ±10% 0402 Multilayer Ceramic Capacitors MLCC - SMD/SMT ROHS"
+		(property "Description" "16V 470nF X7R ±10% 0402 Multilayer Ceramic Capacitors MLCC - SMD/SMT ROHS"
 			(at 118.11 64.77 0)
 			(hide yes)
@@
 			)
 		)
+		(property "LCSC Part #" "C492401"
+			(at 106.68 152.4 0)
+			(hide yes)
+			(show_name no)
+			(do_not_autoplace no)
+			(effects
+				(font
+					(size 1.27 1.27)
+				)
+			)
+		)
+		(property "Mfr. Part #" "PZ254V-11-02P"
+			(at 106.68 152.4 0)
+			(hide yes)
+			(show_name no)
+			(do_not_autoplace no)
+			(effects
+				(font
+					(size 1.27 1.27)
+				)
+			)
+		)
 		(pin "1"
 		)
@@
 			)
 		)
-		(property "Datasheet" "https://www.lcsc.com/datasheet/lcsc_datasheet_2206281830_Murata-Electronics-GRT155R71A474KE01D_C711087.pdf"
+		(property "Datasheet" ""
 			(at 99.06 64.77 0)
 			(hide yes)
@@
 			)
 		)
-		(property "Description" "10V 470nF X7R ±10% 0402 Multilayer Ceramic Capacitors MLCC - SMD/SMT ROHS"
+		(property "Description" "16V 470nF X7R ±10% 0402 Multilayer Ceramic Capacitors MLCC - SMD/SMT ROHS"
 			(at 99.06 64.77 0)
 			(hide yes)
@@
 			)
 		)
-		(property "Datasheet" "https://www.lcsc.com/datasheet/lcsc_datasheet_2206281830_Murata-Electronics-GRT155R71A474KE01D_C711087.pdf"
+		(property "Datasheet" ""
 			(at 86.36 64.77 0)
 			(hide yes)
@@
 			)
 		)
-		(property "Description" "10V 470nF X7R ±10% 0402 Multilayer Ceramic Capacitors MLCC - SMD/SMT ROHS"
+		(property "Description" "16V 470nF X7R ±10% 0402 Multilayer Ceramic Capacitors MLCC - SMD/SMT ROHS"
 			(at 86.36 64.77 0)
 			(hide yes)
@@
 			)
 		)
-		(property "Datasheet" "https://www.lcsc.com/datasheet/lcsc_datasheet_1811081617_Murata-Electronics-GRM155R61A475KEAAD_C77004.pdf"
+		(property "Datasheet" ""
 			(at 163.83 64.77 0)
 			(hide yes)
@@
 			)
 		)
-		(property "Datasheet" "https://www.lcsc.com/datasheet/lcsc_datasheet_2206281830_Murata-Electronics-GRT155R71A474KE01D_C711087.pdf"
+		(property "Datasheet" ""
 			(at 125.73 64.77 0)
 			(hide yes)
@@
 			)
 		)
-		(property "Description" "10V 470nF X7R ±10% 0402 Multilayer Ceramic Capacitors MLCC - SMD/SMT ROHS"
+		(property "Description" "16V 470nF X7R ±10% 0402 Multilayer Ceramic Capacitors MLCC - SMD/SMT ROHS"
 			(at 125.73 64.77 0)
 			(hide yes)
@@
 			)
 		)
-		(property "Datasheet" "https://www.lcsc.com/datasheet/lcsc_datasheet_2309201533_Walsin-Tech-Corp-0402B103K100CT_C3840241.pdf"
+		(property "Datasheet" ""
 			(at 87.63 146.05 0)
 			(hide yes)
@@
 			)
 		)
-		(property "Description" "10V 100nF X7R ±10% 0402 Multilayer Ceramic Capacitors MLCC - SMD/SMT ROHS"
+		(property "Description" "50V 100nF X7R ±10% 0402 Multilayer Ceramic Capacitors MLCC - SMD/SMT ROHS"
 			(at 87.63 146.05 0)
 			(hide yes)
@@
 			)
 		)
-		(property "Datasheet" "https://www.lcsc.com/datasheet/lcsc_datasheet_1811081617_Murata-Electronics-GRM155R61A475KEAAD_C77004.pdf"
+		(property "Datasheet" ""
 			(at 153.67 64.77 0)
 			(hide yes)
