File: RASBB/Hardware/Rev.C/Design/FPGA1_DDR3.kicad_sch (KiCad schematic)
At the start: 32 parts, among them IC9 MT41K256M16TW-107_P

Commit message: Draft AC
Parts:
- C365, C366, C98: LCSC Part # C913474 -> C7281848; Mfr. Part # GRM188Z71A475KE15D -> GMK107BBJ475KA-T
- IC9: value MT41K256M16TW-107_P -> MT41K128M16JT-107:K; LCSC Part # (none) -> C2841151; Mfr. Part # MT41K256M16TW-107:P -> MT41K128M16JT-107:K
