File: RASBB/Hardware/Rev.C/Design/FPGA2_BANK0.kicad_sch (KiCad schematic)
At the start: 16 parts, among them J15 Conn_01x06_Socket, U11 XC7A100T-CSG324

Commit message: Draft AC
Parts:
- added R206: 1.5K, Resistor_SMD:R_0402_1005Metric, symbol Device:R
- added R207: 4K7, Resistor_SMD:R_0402_1005Metric, symbol Device:R_Small
- R160, R161, R162, R163: value 100 -> 49.9; LCSC Part # C163808 -> C4229190; Mfr. Part # WR04X1000FTL -> RMCF0402FT49R9
Connections:
- net FPGA2_DONE: now also R206.2
- net FPGA2_INIT: now also R207.2
- net VCCO_0: now also R206.1, R207.1
Other:
- moved on the sheet: D16, R103, R56
