File: RASBB/Hardware/Rev.C/Design/FPGA2_BANK14-15.kicad_sch (KiCad schematic)
At the start: 20 parts, among them U11 XC7A100T-CSG324

Commit message: Draft AC
Connections:
- net FPGA2_B14_L16: now reaches U11.L16 (IO_L3N_T0_DQS_EMCCLK_14)
- net F2_B15_K13: no longer names the net of U11.K13 (IO_L17P_T2_A26_15)
- net F2_B15_K15: no longer names the net of U11.K15 (IO_L24P_T3_RS1_15)
- no-connect marks 0 -> 11
