File: RASBB/Hardware/Rev.C/Design/FPGA2_BANK16-34.kicad_sch (KiCad schematic)
At the start: 11 parts, among them U11 XC7A100T-CSG324

Commit message: Draft AC
Parts:
- C312: Mfr. Part # GRM155R61A475KEAAD -> GRM155R61A475KEAAD
Connections:
- no-connect marks 0 -> 11
