File: RASBB/Hardware/Rev.C/Design/FPGA2_BANK35.kicad_sch (KiCad schematic)
At the start: 14 parts, among them J18 Conn_01x02_Pin, U11 XC7A100T-CSG324, X4 OT2EL4C4JI-111OLP-50M

Commit message: Draft AC
Parts:
- J18: LCSC Part # (none) -> C492401; Mfr. Part # (none) -> PZ254V-11-02P
- X4: Mfr. Part # (none) -> OT2EL4C4JI-111OLP-50M
Connections:
- net F2_B35_J2: now reaches U11.J2 (IO_L22N_T3_35)
- no-connect marks 0 -> 21
