File: RASBB/Hardware/Rev.C/Design/HDMI.kicad_sch (KiCad schematic)
At the start: 5 parts, among them IC11 TPD12S016PWR, J3 HDMI-001A

Commit message: Draft AC
Parts:
- IC11: LCSC Part #  C201665 -> (none)
- J3: LCSC Part #  C41347845 -> (none)
Other:
- moved on the sheet: J3

Commit message: Modified Based on Findings -Draft
Parts:
- added C240, C286, C288, C309, C318, C319, C320, C321: 100nF, Capacitor_SMD:C_0402_1005Metric, symbol Device:C_Small
- added R212, R213, R214, R215, R216, R217, R218, R219: 270, Resistor_SMD:R_0402_1005Metric, symbol Device:R
Connections:
- net +3V3: now also R212.2, R213.2, R214.2, R215.2, R216.2, R217.2, R218.2, R219.2
- net HDMI_CLK_N: now also C319.1, R219.1; no longer J3.12 (TMDS_CK-)
- net HDMI_CLK_P: now also C318.1, R218.1; no longer J3.10 (TMDS_CK+)
- net HDMI_D0_N: now also C309.1, R217.1; no longer J3.9 (TMDS_D0-)
- net HDMI_D0_P: now also C288.1, R216.1; no longer J3.7 (TMDS_D0+)
- net HDMI_D1_N: now also C286.1, R215.1; no longer J3.6 (TMDS_D1-)
- net HDMI_D1_P: now also C240.1, R214.1; no longer J3.4 (TMDS_D1+)
- net HDMI_D2_N: now also C321.1, R213.1; no longer J3.3 (TMDS_D2-)
- net HDMI_D2_P: now also C320.1, R212.1; no longer J3.1 (TMDS_D2+)
- new net TMDS_CK_N: C319.2, J3.12 (TMDS_CK-)
- new net TMDS_CK_P: C318.2, J3.10 (TMDS_CK+)
- new net TMDS_D0_N: C309.2, J3.9 (TMDS_D0-)
- new net TMDS_D0_P: C288.2, J3.7 (TMDS_D0+)
- new net TMDS_D1_N: C286.2, J3.6 (TMDS_D1-)
- new net TMDS_D1_P: C240.2, J3.4 (TMDS_D1+)
- new net TMDS_D2_N: C321.2, J3.3 (TMDS_D2-)
- new net TMDS_D2_P: C320.2, J3.1 (TMDS_D2+)
Other:
- moved on the sheet: J3
