File: RASBB/Hardware/Rev.C/Design/Interconnect.kicad_sch (KiCad schematic)
At the start: 13 parts, among them J5 FH12-50S-0.5SV

Commit message: Draft AC
Parts:
- J5: LCSC Part # (none) -> C597991; Mfr. Part # (none) -> FH12-50S-0.5SVA(54)
- RN1, RN10, RN2, RN3, RN4, RN5, RN6, RN7, RN8, RN9: LCSC Part # (none) -> C1731024; Mfr. Part # (none) -> CAY10-330J4LF
