File: RASBB/Hardware/Rev.C/Design/PCIE.kicad_sch (KiCad schematic)
At the start: 3 parts, among them J17 Conn_01x02_Pin, J4 X3157WS-98-9TV30

Commit message: Draft AC
Parts:
- added R208, R209: 0, Resistor_SMD:R_1206_3216Metric, symbol Device:R
- J17: LCSC Part # (none) -> C492401; Mfr. Part # (none) -> PZ254V-11-02P
- J4: LCSC Part #  C5711253 -> (none)
- R185: Mfr. Part # (none) -> 1206W4F0000T5E
Connections:
- net +12V: now also R209.2
- net at J4.A01: now also J4.A02, J4.A03, J4.B01, J4.B02, J4.B03, R208.1, R209.1
- new net +5V: R208.2

Commit message: Modified Based on Findings -Draft
Parts:
- R208: now fitted
Connections:
- net GND: now also J4.A32, J4.A33, J4.B10, J4.B11
Changed lines of the file:
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@@
 	(title_block
 		(title "RASBB")
-		(date "2026-07-25")
+		(date "2026-09-20")
 		(rev "C")
 		(company "Mina Daneshpajouh")
@@
 	(wire
 		(pts
+			(xy 113.03 71.12) (xy 121.92 71.12)
+		)
+		(stroke
+			(width 0)
+			(type default)
+		)
+	)
+	(wire
+		(pts
 			(xy 121.92 142.24) (xy 113.03 142.24)
 		)
@@
 	(wire
 		(pts
+			(xy 78.74 129.54) (xy 87.63 129.54)
+		)
+		(stroke
+			(width 0)
+			(type default)
+		)
+	)
+	(wire
+		(pts
 			(xy 113.03 78.74) (xy 121.92 78.74)
 		)
@@
 	(wire
 		(pts
+			(xy 78.74 127) (xy 87.63 127)
+		)
+		(stroke
+			(width 0)
+			(type default)
+		)
+	)
+	(wire
+		(pts
 			(xy 78.74 154.94) (xy 87.63 154.94)
 		)
@@
 		(pts
 			(xy 121.92 132.08) (xy 113.03 132.08)
+		)
+		(stroke
+			(width 0)
+			(type default)
+		)
+	)
+	(wire
+		(pts
+			(xy 113.03 73.66) (xy 121.92 73.66)
 		)
 		(stroke
@@
 	)
 	(label "GND"
+		(at 78.74 127 0)
+		(effects
+			(font
+				(size 1.27 1.27)
+			)
+			(justify left bottom)
+		)
+	)
+	(label "GND"
 		(at 121.92 165.1 180)
 		(effects
@@
 		)
 	)
+	(label "GND"
+		(at 121.92 73.66 180)
+		(effects
+			(font
+				(size 1.27 1.27)
+			)
+			(justify right bottom)
+		)
+	)
 	(label "RX7_N"
 		(at 121.92 116.84 180)
@@
 	)
 	(label "GND"
+		(at 78.74 129.54 0)
+		(effects
+			(font
+				(size 1.27 1.27)
+			)
+			(justify left bottom)
+		)
+	)
+	(label "GND"
 		(at 121.92 127 180)
 		(effects
@@
 	(label "GND"
 		(at 121.92 147.32 180)
+		(effects
+			(font
+				(size 1.27 1.27)
+			)
+			(justify right bottom)
+		)
+	)
+	(label "GND"
+		(at 121.92 71.12 180)
 		(effects
 			(font
@@
 		(on_board yes)
 		(in_pos_files yes)
-		(dnp yes)
+		(dnp no)
 		(property "Reference" "R208"
 			(at 131.826 45.974 90)
@@
 		(in_pos_files yes)
 		(dnp no)
+		(fields_autoplaced yes)
 		(property "Reference" "J4"
-			(at 99.822 177.038 0)
+			(at 100.33 175.26 0)
 			(show_name no)
 			(do_not_autoplace no)
@@
 		)
 		(property "Value" "X3157WS-98-9TV30"
-			(at 99.822 179.578 0)
-			(show_name no)
-			(do_not_autoplace no)
+			(at 100.33 177.8 0)
+			(show_name no)
+			(do_not_autoplace no)
