File: RASBB/Hardware/Rev.C/Design/POQWE.kicad_sch (KiCad schematic)
At the start: 117 parts, among them IC1 RT6365GSP, IC2 TPS56528DDAR, IC3 TPS563201DDCR, IC4 TPS56528DDAR, J1 PJ-002AH-SMT-TR, U1 SZMMSZ4702T1G, U2 SI2324DS-T1-GE3, U3 SIC453ED-T1-GE3, U4 JW5026

Commit message: Draft AC
Parts:
- C11, C38, C39, C40, C50, C51: LCSC Part # C3840241 -> C301927; Mfr. Part # 0402B103K100CT -> 0402B103K500CT
- C17: LCSC Part # C178582 -> C178581; Mfr. Part # EEE-FP1V331AP -> EEE-FP1V330AP
- C29: LCSC Part # C913474 -> C7281848; Mfr. Part # GRM155R61A475KEAAD -> GMK107BBJ475KA-T
- C3, C7: Mfr. Part # (none) -> CGA0603X7R103K101JT
- D1: LCSC Part #  C3024223 -> (none)
- D2, D3: LCSC Part #  C6000165 -> (none)
- F2: Mfr. Part # BSMD1812-150-33V -> BSMD1812-200-30V
- IC1: LCSC Part #  C3024482 -> (none)
- IC3: LCSC Part #  C116592 -> (none)
- L1: LCSC Part #  C2595948 -> (none)
- L3: LCSC Part #  C845083 -> (none)
- L4, L5, L6: LCSC Part #  C845037 -> (none)
- R31: LCSC Part # C384380 -> C137924; Mfr. Part # CRCW04023R30FKEDC -> RC0402JR-07120KL
Connections:
- net +12V: no longer F2.2
- net GND: now also U2.2 (S); no longer U2.3 (D)
- net RTN: now also U2.3 (D); no longer U2.2 (S)
- net at C16.1, D2.1, D3.1: now also F2.2; no longer F2.1
Other:
- moved on the sheet: F2, U2

Commit message: Modified Based on Findings -Draft
Parts:
- removed D17, D18, D19: A-SP192DGHC-C01-4T, LED_SMD:LED_0603_1608Metric, symbol Device:LED
- removed R128, R129, R130: 715, Resistor_SMD:R_0402_1005Metric, symbol Device:R_Small
- added R211: 0.005, Resistor_SMD:R_2512_6332Metric, symbol Device:R_Small
- C4: value 10uF/100V -> 10uF
- R35, R42, R49: now fitted
Connections:
- net +12V: now also R211.1
- net GND: now also U2.3 (D); no longer U2.2 (S)
- net RTN: now also U2.2 (S); no longer U2.3 (D)
- net at F2.1: now also R211.2
Other:
- moved on the sheet: C4, U2
