File: RASBB/Hardware/Rev.C/Design/RASBB.kicad_sch (KiCad schematic)
At the start: 71 parts, among them J20 Conn_01x02_Pin, SW1 435451019820, SW2 435451019820, U5 TLV9001DBVR

Commit message: Draft AC
Parts:
- added C240, C286, C288, C309, C318, C319, C320, C321: 100nF, Capacitor_SMD:C_0402_1005Metric, symbol Device:C_Small
- C270: LCSC Part # (none) -> C152814; Mfr. Part # (none) -> 0402B104K500CT
- C271, R151: now fitted
- C272: LCSC Part # (none) -> C1531; Mfr. Part # (none) -> 0402B222K500NT
- J20: LCSC Part # (none) -> C492401; Mfr. Part # (none) -> PZ254V-11-02P
- R10: LCSC Part #  C163826 -> (none)
- R168, R169, R170, R171, R172, R173, R174, R175, R176, R177, R178, R179, R180, R181, R182, R183, R184: footprint Resistor_SMD:R_0201_0603Metric -> Resistor_SMD:R_0402_1005Metric
- R195, R200, R201: LCSC Part # (none) -> C25804; Mfr. Part # (none) -> 0603WAF1002T5E
- SW1, SW2: footprint Switch_SMD_Wurth:SW_Wurth_WS-TASV_435451019820 -> RASBB:435451019820; Mfr. Part # (none) -> 435451019820
- U5: Mfr. Part # (none) -> TLV9001QDBVRQ1
Connections:
- net FPGA-01/F1_B15_A13: now also C320.1
- net FPGA-01/F1_B15_A14: now also C321.1
- net FPGA-01/F1_B15_A15: now also C288.1
- net FPGA-01/F1_B15_A16: now also C309.1
- net FPGA-01/F1_B15_A18: now also C286.1
- net FPGA-01/F1_B15_B16: now also C318.1
- net FPGA-01/F1_B15_B17: now also C319.1
- net FPGA-01/F1_B15_B18: now also C240.1
- net GND: now also J20.1 (Pin_1), SW1.2, SW1.5 (GND), SW2.2, SW2.5 (GND); no longer SW1.GND, SW2.GND
- net FPGA1_RESET: now reaches SW1.4
- net FPGA2_RESET: now reaches SW2.4
- net FPGA-02/F2_B35_J2: now reaches R195.1
- new net HDMI/HDMI_CLK_N: C321.2
- new net HDMI/HDMI_CLK_P: C320.2
- new net HDMI/HDMI_D0_N: C319.2
- new net HDMI/HDMI_D0_P: C318.2
- new net HDMI/HDMI_D1_N: C309.2
- new net HDMI/HDMI_D1_P: C288.2
- new net HDMI/HDMI_D2_N: C286.2
- new net HDMI/HDMI_D2_P: C240.2
Other:
- sheet Ethernet_uC ports: added CLK_OVR_ETH; removed none
- sheet FPGA-01 ports: added F1_B15_F18, F1_B15_G18; removed none
- sheet FPGA-02 ports: added F2_B14_L16, F2_B35_J2; removed F2_B15_K13, F2_B15_K15
- sheet uController ports: added uC_PC2, uC_PE0; removed none
- note removed: "FPG1"
- note removed: "from FPGA2"

Commit message: Modified Based on Findings -Draft
Parts:
- removed C240, C286, C288, C309, C318, C319, C320, C321: 100nF, Capacitor_SMD:C_0402_1005Metric, symbol Device:C_Small
- R150: now fitted
Other:
- sheet Inteconnect renamed Interconnect (page 11)
