File: RASBB/Hardware/Rev.C/Design/RF_Transceiver.kicad_sch (KiCad schematic)
At the start: 21 parts, among them IC13 SX1280IMLTRT, J11 Conn_Coaxial, Y2 XC21M4-52.000-F10NNHPL

Commit message: Draft AC
Parts:
- C150, C151: LCSC Part # C3840241 -> C301927; Mfr. Part # 0402B103K100CT -> 0402B103K500CT
- FB3: LCSC Part #  C710334 -> (none)
- L10: LCSC Part #  C317668 -> (none)
- L9: LCSC Part #  C433005 -> (none)
Changed lines of the file:
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@@
 			)
 		)
-		(property "Datasheet" "https://www.lcsc.com/datasheet/lcsc_datasheet_2309201533_Walsin-Tech-Corp-0402B103K100CT_C3840241.pdf"
+		(property "Datasheet" ""
 			(at 119.38 119.38 0)
 			(hide yes)
@@
 			)
 		)
-		(property "Description" "10V 100nF X7R ±10% 0402 Multilayer Ceramic Capacitors MLCC - SMD/SMT ROHS"
+		(property "Description" "50V 100nF X7R ±10% 0402 Multilayer Ceramic Capacitors MLCC - SMD/SMT ROHS"
 			(at 119.38 119.38 0)
 			(hide yes)
@@
 			)
 		)
-		(property "Datasheet" "https://www.lcsc.com/datasheet/lcsc_datasheet_2309201533_Walsin-Tech-Corp-0402B103K100CT_C3840241.pdf"
+		(property "Datasheet" ""
 			(at 149.86 93.98 0)
 			(hide yes)
@@
 			)
 		)
-		(property "Description" "10V 100nF X7R ±10% 0402 Multilayer Ceramic Capacitors MLCC - SMD/SMT ROHS"
+		(property "Description" "50V 100nF X7R ±10% 0402 Multilayer Ceramic Capacitors MLCC - SMD/SMT ROHS"
 			(at 149.86 93.98 0)
 			(hide yes)
@@
 			)
 		)
-		(property "Description" "Inductor"
+		(property "Description" "3nH 800mA ±0.1nH 0402 High Frequency / RF Inductors - Surface Mount ROHS"
 			(at 157.48 53.34 0)
 			(hide yes)
@@
 			)
 		)
-		(property "LCSC Part # " "C433005"
+		(property "LCSC Part # " ""
 			(at 157.48 53.34 90)
 			(hide yes)
@@
 			)
 		)
-		(property "Datasheet" "https://www.lcsc.com/datasheet/lcsc_datasheet_2409272300_YAGEO-CC0402KRX7R6BB103_C541371.pdf"
+		(property "Datasheet" ""
 			(at 95.25 73.66 0)
 			(hide yes)
@@
 			)
 		)
-		(property "Description" "10V 10nF X7R ±10% 0402 Multilayer Ceramic Capacitors MLCC - SMD/SMT ROHS"
+		(property "Description" "50V 10nF X7R ±10% 0402 Multilayer Ceramic Capacitors MLCC - SMD/SMT ROHS"
 			(at 95.25 73.66 0)
 			(hide yes)
@@
 			)
 		)
-		(property "Mfr. Part #" "0402B103K100CT"
+		(property "Mfr. Part #" "0402B103K500CT"
 			(at 95.25 73.66 0)
 			(hide yes)
@@
 			)
 		)
-		(property "LCSC Part #" "C3840241"
+		(property "LCSC Part #" "C301927"
 			(at 95.25 73.66 0)
 			(hide yes)
@@
 			)
 		)
-		(property "Datasheet" "https://www.lcsc.com/datasheet/lcsc_datasheet_2206281830_Murata-Electronics-GRT155R71A474KE01D_C711087.pdf"
+		(property "Datasheet" ""
 			(at 135.89 118.11 0)
 			(hide yes)
@@
 			)
 		)
-		(property "Description" "10V 470nF X7R ±10% 0402 Multilayer Ceramic Capacitors MLCC - SMD/SMT ROHS"
+		(property "Description" "16V 470nF X7R ±10% 0402 Multilayer Ceramic Capacitors MLCC - SMD/SMT ROHS"
 			(at 135.89 118.11 0)
 			(hide yes)
@@
 			)
 		)
-		(property "Datasheet" "https://www.lcsc.com/datasheet/lcsc_datasheet_2409272300_YAGEO-CC0402KRX7R6BB103_C541371.pdf"
+		(property "Datasheet" ""
 			(at 86.36 76.2 0)
 			(hide yes)
@@
 			)
 		)
-		(property "Description" "10V 10nF X7R ±10% 0402 Multilayer Ceramic Capacitors MLCC - SMD/SMT ROHS"
+		(property "Description" "50V 10nF X7R ±10% 0402 Multilayer Ceramic Capacitors MLCC - SMD/SMT ROHS"
 			(at 86.36 76.2 0)
 			(hide yes)
@@
 			)
 		)
-		(property "Mfr. Part #" "0402B103K100CT"
+		(property "Mfr. Part #" "0402B103K500CT"
 			(at 86.36 76.2 0)
 			(hide yes)
@@
 			)
 		)
-		(property "LCSC Part #" "C3840241"
+		(property "LCSC Part #" "C301927"
 			(at 86.36 76.2 0)
 			(hide yes)
@@
 			)
 		)
-		(property "Datasheet" "https://www.lcsc.com/datasheet/lcsc_datasheet_2309201533_Walsin-Tech-Corp-0402B103K100CT_C3840241.pdf"
+		(property "Datasheet" ""
 			(at 68.58 134.62 0)
 			(hide yes)
@@
 			)
 		)
-		(property "Description" "10V 100nF X7R ±10% 0402 Multilayer Ceramic Capacitors MLCC - SMD/SMT ROHS"
+		(property "Description" "50V 100nF X7R ±10% 0402 Multilayer Ceramic Capacitors MLCC - SMD/SMT ROHS"
 			(at 68.58 134.62 0)
 			(hide yes)
@@
 			)
 		)
-		(property "LCSC Part # " "C710334"
+		(property "LCSC Part # " ""
 			(at 25.4 128.27 0)
 			(hide yes)
@@
 			)
 		)
-		(property "LCSC Part # " "C317668"
+		(property "LCSC Part # " ""
 			(at 173.99 53.34 90)
 			(hide yes)
