File: RASBB/Hardware/Rev.C/Design/uController.kicad_sch (KiCad schematic)
At the start: 61 parts, among them IC12 STM32H743VGT6, J10 ZX-PZ1.27-2-5PWZ, J7 USB_C_Receptacle, J8 ZX-PZ1.27-2-5PWZ, J9 KF2EDGR-3.5-2P, Q1 DMN6075S, U6 CH340E, U7 AHT20, Y1 X503220MSB2GI

Commit message: Draft AC
Parts:
- added C276, C323: 100nF, Capacitor_SMD:C_0402_1005Metric, symbol Device:C_Small
- added C279: 4.7uF, Capacitor_SMD:C_0603_1608Metric, symbol Device:C_Small
- added D27: SMAJ33A, DIOM5026X229N, symbol RASBB_Library:SMAJ33A
- added TP24, TP25: TestPoint, TestPoint:TestPoint_Pad_D1.0mm, symbol Connector:TestPoint
- C127, C128: LCSC Part # C913474 -> C7281848; Mfr. Part # GRM188Z71A475KE15D -> GMK107BBJ475KA-T
- C139, C140: footprint Capacitor_SMD:C_0603_1608Metric -> Capacitor_SMD:C_0402_1005Metric
- F1: Mfr. Part # (none) -> BSMD1812-150-33V
- FB1, FB2: LCSC Part #  C710334 -> (none)
- IC12: LCSC Part #  C730183 -> (none)
- J10, J8: LCSC Part #  C41370773 -> (none)
- R101, R114, R115, R116, R117, R118, R119, R120: LCSC Part #  C163826 -> (none)
Connections:
- net +3V3: now also C323.1
- net FPGA1_DONE: now also IC12.22 (PA0); no longer IC12.20 (VREF+)
- net GND: now also C276.2, C279.2, C323.2, D27.2
- net uC_PC2: now reaches IC12.17 (PC2_C)
- net uC_PE0: now reaches IC12.97 (PE0)
- net at D6.1 (K), F1.1, Q1.3 (D): now also D27.1
- net PD0_DEBUG: no longer names the net of IC12.81 (PD0)
- net PD0_DEBUG: now also TP24.1
- net PD10_DEBUG: no longer names the net of IC12.57 (PD10)
- net PD10_DEBUG: now also TP25.1
- new net: C276.1, C279.1, IC12.20 (VREF+)
- no-connect marks 0 -> 1
Other:
- moved on the sheet: D6, F1, J9

Commit message: Modified Based on Findings -Draft
Parts:
- added C324: 100nF, Capacitor_SMD:C_0402_1005Metric, symbol Device:C_Small
Connections:
- net +3V3: no longer J10.2
- net DBG_JTCK_SWCLK: now also J10.4; no longer J10.8, J10.9
- net DBG_JTDI: now also J10.8; no longer J10.5
- net DBG_JTDO_SWO: now also R115.1; no longer R119.1
- net DBG_JTMS_SWDIO: now also J10.2, R116.1; no longer J10.7, R115.1
- net GND: now also J10.3, J10.5, J10.9, C324.2; no longer J10.10
- net uC_NRST: now also J10.10, R119.1, C324.1; no longer J10.3, R116.1
- no-connect marks 1 -> 2
Other:
- moved on the sheet: R119, R120
